File: POVwatch_1.sch (EAGLE design)
At the start: 48 parts, among them Q1 S8050, U1 ATMEGA168P-AU, U2 ADXL345, U3 MCP6001-SOT23, U4 APDS-9008, U5 TP4056, U6 3.3V, Y1 7.3728MHz

Commit message: This is POVwatch 1.0.1 (bugs fixed)
Parts:
- added R1: 10kΩ, MyLibrary:RES-0603
- added TS1: TS-3035, MyLibrary:TS-3035
- CO3: value 4.7μF -> 2.2μF
- CX1, CX2: value 22μF -> 22pF
Connections:
- new net BUTTON: R1.1, TS1.2, U1.PD5(T1)
- net GND: now also R1.2, U1.GND@1, U1.GND@2, U1.GND@3, U2.GND@1, U2.GND@2, U2.GND@3; no longer U1.GND1, U1.GND2, U1.GND3, U2.GND1, U2.GND2, U2.GND3
- net VDD_3V3: now also TS1.1, U1.VCC@1, U1.VCC@2; no longer U1.VCC1, U1.VCC2
Other:
- note added: "Heart Rate Sensor"
- note added: "in AVR, so we don't need to add RSDA and RSCL."
- note removed: "Pulse Sensor"
- note removed: "in AVR, so we don't need to add RSDA and RSCl."
Changed lines of the file:
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@@
 <part name="SUPPLY12" library="MyLibrary" deviceset="GND" device=""/>
 <part name="Y1" library="MyLibrary" deviceset="XTAL" device="-5032" value="7.3728MHz"/>
-<part name="CX1" library="MyLibrary" deviceset="CAP" device="-0603" value="22μF"/>
-<part name="CX2" library="MyLibrary" deviceset="CAP" device="-0603" value="22μF"/>
+<part name="CX1" library="MyLibrary" deviceset="CAP" device="-0603" value="22pF"/>
+<part name="CX2" library="MyLibrary" deviceset="CAP" device="-0603" value="22pF"/>
 <part name="SUPPLY14" library="MyLibrary" deviceset="GND" device=""/>
 <part name="CAVCC" library="MyLibrary" deviceset="CAP" device="-0603" value="100nF"/>
@@
 <part name="CO1" library="MyLibrary" deviceset="CAP" device="-0603" value="4.7μF"/>
 <part name="CO2" library="MyLibrary" deviceset="CAP" device="-0603" value="4.7μF"/>
-<part name="CO3" library="MyLibrary" deviceset="CAP" device="-0603" value="4.7μF"/>
+<part name="CO3" library="MyLibrary" deviceset="CAP" device="-0603" value="2.2μF"/>
 <part name="CO4" library="MyLibrary" deviceset="CAP" device="-0603" value="4.7μF"/>
 <part name="SUPPLY2" library="MyLibrary" deviceset="GND" device=""/>
@@
 <part name="RP1" library="MyLibrary" deviceset="RP" device="-0603" value="470Ω"/>
 <part name="RP2" library="MyLibrary" deviceset="RP" device="-0603" value="470Ω"/>
+<part name="TS1" library="MyLibrary" deviceset="TS" device="-3035" value="TS-3035"/>
+<part name="R1" library="MyLibrary" deviceset="RES" device="-0603" value="10kΩ"/>
+<part name="SUPPLY13" library="MyLibrary" deviceset="GND" device=""/>
+<part name="SUPPLY27" library="MyLibrary" deviceset="VDD_3V3" device=""/>
 </parts>
 <sheets>
@@
 <text x="-55.88" y="50.8" size="2.54" layer="97" font="vector">MCU Central Controller</text>
 <text x="-134.62" y="0" size="2.54" layer="97" font="vector">Acceleration Sensor</text>
-<text x="-182.88" y="50.8" size="2.54" layer="95" font="vector">Pulse Sensor</text>
+<text x="-182.88" y="50.8" size="2.54" layer="95" font="vector">Heart Rate Sensor</text>
 <wire x1="-193.04" y1="60.96" x2="-193.04" y2="-43.18" width="0.4064" layer="97" style="longdash"/>
 <wire x1="-193.04" y1="-43.18" x2="-139.7" y2="-43.18" width="0.4064" layer="97" style="longdash"/>
@@
 <text x="60.96" y="-2.54" size="2.54" layer="97" font="vector">Display LEDs</text>
 <text x="-134.62" y="7.62" size="1.27" layer="97" font="vector">There are internal pull-up resistors</text>
-<text x="-134.62" y="5.08" size="1.27" layer="97" font="vector">in AVR, so we don't need to add RSDA and RSCl.</text>
+<text x="-134.62" y="5.08" size="1.27" layer="97" font="vector">in AVR, so we don't need to add RSDA and RSCL.</text>
 </plain>
 <instances>
@@
 <instance part="SUPPLY12" gate="GND" x="-40.64" y="0"/>
 <instance part="Y1" gate="A" x="-40.64" y="15.24" smashed="yes">
-<attribute name="NAME" x="-36.83" y="17.78" size="1.778" layer="95" align="center-left"/>
-<attribute name="VALUE" x="-39.37" y="8.89" size="1.778" layer="96" align="center-left"/>
+<attribute name="NAME" x="-34.29" y="8.89" size="1.778" layer="95" rot="R180" align="center-left"/>
+<attribute name="VALUE" x="-34.29" y="6.35" size="1.778" layer="96" rot="R180" align="center-left"/>
 </instance>
 <instance part="CX1" gate="A" x="-45.72" y="20.32" smashed="yes" rot="R90">
@@
 <instance part="RCHRG" gate="A" x="86.36" y="30.48"/>
 <instance part="CBAT" gate="A" x="127" y="35.56"/>
-<instance part="LI-ION" gate="A" x="142.24" y="35.56" rot="R90"/>
+<instance part="LI-ION" gate="A" x="142.24" y="35.56" smashed="yes" rot="R90">
+<attribute name="NAME" x="147.955" y="36.83" size="1.778" layer="95" rot="R270"/>
+<attribute name="VALUE" x="149.86" y="36.83" size="1.778" layer="96" rot="R270"/>
+</instance>
 <instance part="SUPPLY17" gate="GND" x="106.68" y="12.7"/>
 <instance part="SUPPLY18" gate="GND" x="127" y="27.94"/>
@@
 <instance part="SUPPLY25" gate="GND" x="177.8" y="-27.94"/>
 <instance part="SUPPLY26" gate="VDD_3V3" x="193.04" y="-15.24" rot="R270"/>
-<instance part="RTRIG" gate="A" x="-172.72" y="-15.24"/>
+<instance part="RTRIG" gate="A" x="-172.72" y="-15.24" smashed="yes">
+<attribute name="NAME" x="-175.26" y="-18.796" size="1.778" layer="95"/>
+<attribute name="VALUE" x="-175.26" y="-21.336" size="1.778" layer="96"/>
+</instance>
 <instance part="DDIS1" gate="A" x="96.52" y="-12.7" smashed="yes" rot="R90">
 <attribute name="NAME" x="104.14" y="-12.7" size="1.778" layer="95"/>
@@
 <instance part="U6" gate="P" x="177.8" y="33.02"/>
 <instance part="SUPPLY29" gate="GND" x="177.8" y="17.78"/>
-<instance part="CVIN" gate="A" x="165.1" y="25.4"/>
-<instance part="CVOUT" gate="A" x="187.96" y="25.4"/>
+<instance part="CVIN" gate="A" x="165.1" y="25.4" smashed="yes">
+<attribute name="NAME" x="161.036" y="25.019" size="1.778" layer="95" rot="R180"/>
+<attribute name="VALUE" x="161.036" y="22.479" size="1.778" layer="96" rot="R180"/>
+</instance>
+<instance part="CVOUT" gate="A" x="187.96" y="25.4" smashed="yes">
+<attribute name="NAME" x="192.024" y="23.241" size="1.778" layer="95"/>
+<attribute name="VALUE" x="192.024" y="20.701" size="1.778" layer="96"/>
+</instance>
 <instance part="RP1" gate="A" x="81.28" y="-10.16" smashed="yes" rot="R180">
 <attribute name="NAME" x="83.82" y="-10.16" size="1.778" layer="95"/>
@@
 <attribute name="VALUE" x="89.916" y="-27.94" size="1.778" layer="96"/>
 </instance>
+<instance part="TS1" gate="A" x="27.94" y="38.1" rot="R90"/>
+<instance part="R1" gate="A" x="40.64" y="38.1" rot="R180"/>
+<instance part="SUPPLY13" gate="GND" x="48.26" y="38.1" rot="R90"/>
+<instance part="SUPPLY27" gate="VDD_3V3" x="17.78" y="38.1" rot="R90"/>
 </instances>
 <busses>
@@
 <pinref part="SUPPLY6" gate="VDD_3V3" pin="VDD_3V3"/>
 <wire x1="0" y1="43.18" x2="5.08" y2="43.18" width="0.1524" layer="91"/>
-<pinref part="U1" gate="P" pin="VCC2"/>
+<pinref part="U1" gate="P" pin="VCC@2"/>
 <wire x1="5.08" y1="43.18" x2="5.08" y2="33.02" width="0.1524" layer="91"/>
 <junction x="0" y="43.18"/>
-<pinref part="U1" gate="P" pin="VCC1"/>
+<pinref part="U1" gate="P" pin="VCC@1"/>
 <wire x1="0" y1="43.18" x2="0" y2="33.02" width="0.1524" layer="91"/>
 <pinref part="LAVCC" gate="A" pin="2"/>
@@
 <junction x="187.96" y="33.02"/>
 </segment>
+<segment>
+<pinref part="TS1" gate="A" pin="1"/>
+<pinref part="SUPPLY27" gate="VDD_3V3" pin="VDD_3V3"/>
+</segment>
 </net>
 <net name="GND" class="0">
 <segment>
-<pinref part="U1" gate="P" pin="GND2"/>
+<pinref part="U1" gate="P" pin="GND@2"/>
 <pinref part="SUPPLY7" gate="GND" pin="GND"/>
-<pinref part="U1" gate="P" pin="GND1"/>
+<pinref part="U1" gate="P" pin="GND@1"/>
 <wire x1="-5.08" y1="-30.48" x2="0" y2="-30.48" width="0.1524" layer="91"/>
 <junction x="0" y="-30.48"/>
-<pinref part="U1" gate="P" pin="GND3"/>
+<pinref part="U1" gate="P" pin="GND@3"/>
 <wire x1="0" y1="-30.48" x2="5.08" y2="-30.48" width="0.1524" layer="91"/>
 </segment>
@@
 </segment>
 <segment>
-<pinref part="U2" gate="P" pin="GND2"/>
+<pinref part="U2" gate="P" pin="GND@2"/>
 <pinref part="SUPPLY10" gate="GND" pin="GND"/>
-<pinref part="U2" gate="P" pin="GND1"/>
+<pinref part="U2" gate="P" pin="GND@1"/>
 <wire x1="-116.84" y1="-35.56" x2="-114.3" y2="-35.56" width="0.1524" layer="91"/>
 <junction x="-114.3" y="-35.56"/>
-<pinref part="U2" gate="P" pin="GND3"/>
+<pinref part="U2" gate="P" pin="GND@3"/>
 <wire x1="-114.3" y1="-35.56" x2="-111.76" y2="-35.56" width="0.1524" layer="91"/>
 </segment>
@@
 <wire x1="187.96" y1="20.32" x2="187.96" y2="22.86" width="0.1524" layer="91"/>
 </segment>
+<segment>
+<pinref part="R1" gate="A" pin="2"/>
+<pinref part="SUPPLY13" gate="GND" pin="GND"/>
+</segment>
 </net>
 <net name="SCL" class="0">
@@
 </segment>
 </net>
+<net name="BUTTON" class="0">
+<segment>
+<pinref part="U1" gate="P" pin="PD5(T1)"/>
+<wire x1="35.56" y1="7.62" x2="40.64" y2="7.62" width="0.1524" layer="91"/>
+<label x="40.64" y="7.62" size="1.778" layer="95" font="vector"/>
+</segment>
+<segment>
+<pinref part="TS1" gate="A" pin="2"/>
+<pinref part="R1" gate="A" pin="1"/>
+<wire x1="35.56" y1="38.1" x2="35.56" y2="43.18" width="0.1524" layer="91"/>
+<junction x="35.56" y="38.1"/>
+<label x="35.56" y="43.18" size="1.778" layer="95" font="vector" rot="R90"/>
+</segment>
+</net>

Commit message: This is POVwatch 1.1 (begin)
Parts:
- removed CAVCC: 100nF, MyLibrary:CAP-0603
- removed CVIN: 1μF, MyLibrary:CAP-0603
- removed CX1, CX2: 22pF, MyLibrary:CAP-0603
- removed DSTDBY: GREEN, MyLibrary:LED-0603
- removed LAVCC: 22μH, MyLibrary:IND-0805
- removed R1: 10kΩ, MyLibrary:RES-0603
- removed RDP1, RDP2: 220Ω, MyLibrary:RES-0603
- removed RSTDBY: 1kΩ, MyLibrary:RES-0603
- added FB1, FB2, FB3, FB4: BROAD-STICK, MyLibrary:BROAD-STICK
- added HD3: HEADER1X10, MyLibrary:HEADER1X10
- added JP1: USB-MICRO, MyLibrary:USB-MICRO
- added RDP: 220Ω, MyLibrary:RES-0603
- added RESET: JUMPER-SMD, MyLibrary:JUMPER-SMD
- added U7: CH340E, MyLibrary:CH340E
- HD1: value HEADER1X4-SMD1.25 -> HEADER1X10-FPC0.5; device MyLibrary:HEADER1X4-SMD1.25 -> MyLibrary:HEADER1X10-FPC0.5
- LI-ION: value BATTERY-SMD1.25 -> BATTERY-SMD; device MyLibrary:BATTERY-SMD1.25 -> MyLibrary:BATTERY-SMD
- TS1: value TS-3035 -> TS-P; device MyLibrary:TS-3035 -> MyLibrary:TS-P
- U1: value ATMEGA168P-AU -> ATMEGA168P-QFN32; device MyLibrary:ATMEGA168P-AU -> MyLibrary:ATMEGA168P-QFN32
- U5: value TP4056 -> TP4055; device MyLibrary:TP4056 -> MyLibrary:TP4055
- Y1: device MyLibrary:XTAL-5032 -> MyLibrary:CSTCE
Connections:
- net CHRG renamed !CHRG
- net CHRGR renamed DRCHRG
- net PROGR renamed PROG
- net TRIGR renamed RQTRIG
- removed net AVCC: CAVCC.2, LAVCC.1, U1.AVCC
- removed net BUTTON: R1.1, TS1.2, U1.PD5(T1)
- removed net COLLECT: Q1.C, RDP1.1, RDP2.1
- removed net INT2: U1.PD3(INT1), U2.INT2
- removed net LR1: DP1.C, RDP1.2
- removed net LR2: DP2.C, RDP2.2
- removed net N$22: DDIS1.A, RP1B.2
- removed net N$23: DDIS2.A, RP1C.2
- removed net N$24: DDIS3.A, RP1D.2
- removed net N$25: DDIS4.A, RP2A.2
- removed net N$26: DDIS5.A, RP2B.2
- removed net N$27: DDIS6.A, RP2C.2
- removed net N$28: DDIS7.A, RP2D.2
- removed net N$29: DDIS0.A, RP1A.2
- removed net STDBY: RSTDBY.1, U5.!STDBY
- removed net STDBYR: DSTDBY.C, RSTDBY.2
- removed net VCC: DCHRG.A, DSTDBY.A, HD1.2, U5.CE, U5.VCC
- new net !GND: DDIS0.C, DDIS1.C, DDIS2.C, DDIS3.C, DDIS4.C, DDIS5.C, DDIS6.C, DDIS7.C, HD3.5, HD3.6
- new net GND(CH340E): JP1.GND, U7.GND
- new net HD0: DDIS0.A, HD3.1
- new net HD1: DDIS1.A, HD3.2
- new net HD2: DDIS2.A, HD3.3
- new net HD3: DDIS3.A, HD3.4
- new net HD4: DDIS4.A, HD3.7
- new net HD5: DDIS5.A, HD3.8
- new net HD6: DDIS6.A, HD3.9
- new net HD7: DDIS7.A, HD3.10
- new net INT0: TS1.1, U1.PD2(INT0)
- new net QRP: Q1.E, RDP.2
- new net RDP: DP1.A, DP2.A, RDP.1
- new net RH0: HD1.1, RP1A.2
- new net RH1: HD1.2, RP1B.2
- new net RH2: HD1.3, RP1C.2
- new net RH3: HD1.4, RP1D.2
- new net RH4: HD1.7, RP2A.2
- new net RH5: HD1.8, RP2B.2
- new net RH6: HD1.9, RP2C.2
- new net RH7: HD1.10, RP2D.2
- new net UD+: JP1.D+, U7.UD+
- new net UD-: JP1.D-, U7.UD-
- new net VUSB: DCHRG.A, JP1.VBUS, U5.VCC
- net GND: now also DP1.C, DP2.C, FB1.GND, FB2.GND, FB3.GND, FB4.GND, HD1.5, HD1.6, JP1.SHELL, RESET.1, TS1.2, Y1.2; no longer CAVCC.1, CVIN.2, CX1.1, CX2.1, DDIS0.C, DDIS1.C, DDIS2.C, DDIS3.C, DDIS4.C, DDIS5.C, DDIS6.C, DDIS7.C, HD1.1, Q1.E, R1.2, U5.TEMP
- net INT1: now also U1.PD3(INT1); no longer U1.PD2(INT0)
- net OUT0: now also U1.PC0(ADC0)
- net RESET: now also RESET.2
- net RXD: now also U7.TXD; no longer HD1.3
- net TXD: now also U7.RXD; no longer HD1.4
- net VBAT: no longer CVIN.1
- net VDD_3V3: now also Q1.C, U1.AVCC, U7.V3, U7.VCC; no longer DP1.A, DP2.A, LAVCC.2, TS1.1
- net X1: now also Y1.1; no longer CX1.2, Y1.A
- net X2: now also Y1.3; no longer CX2.2, Y1.B
Other:
- note added: "As the USB cable plugged in, the shell and the"
- note added: "Enable internal pull-up resistors"
- note added: "Ground Only For CH340E Connected, the battery starts to feed power."
- note added: "Internal Pull Up Resistor Here"
- note added: "Short this jumper with"
- note added: "USB to TTL"
- note added: "in AVR to avoid adding RSDA and RSCL."
- note added: "tweezers to reset the MCU."
- note removed: "There are internal pull-up resistors"
- note removed: "USART"
- note removed: "in AVR, so we don't need to add RSDA and RSCL."
- moved on the sheet: CBAT, CVOUT, DCHRG, DDIS0, DDIS1, DDIS2, DDIS3, DDIS4, DDIS5, DDIS6, DDIS7, DP1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
